File: hardware/MT32-DIT-board/MT32-DIT-board.kicad_sch (KiCad schematic)
At the start: 47 parts, among them J1 I2S_CONN, J2 spdif_dit, J3 spdif_wm, T1 PE-65612NL, U1 DIT4192IPW, U2 WM8804

Commit message: M/S pin was not connected due to Kicad terrible grid, fixed
Connections:
- net GNDREF: no longer JP5.2 (B), JP6.2 (B), JP7.2 (B)
- net M/S: now also JP9.1 (A), R10.2
- new net: JP5.2 (B), JP6.2 (B), JP7.2 (B)
Changed lines of the file:
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@@
 	)
 	(junction
+		(at 161.671 78.3955)
+		(diameter 0)
+		(color 0 0 0 0)
+	)
+	(junction
 		(at 213.487 56.515)
 		(diameter 0)
@@
 	)
 	(junction
+		(at 164.846 80.9244)
+		(diameter 0)
+		(color 0 0 0 0)
+	)
+	(junction
 		(at 161.671 96.139)
 		(diameter 0)
@@
 	)
 	(junction
-		(at 175.006 80.899)
-		(diameter 0)
-		(color 0 0 0 0)
-	)
-	(junction
 		(at 121.539 91.44)
 		(diameter 0)
@@
 	)
 	(junction
-		(at 161.671 78.359)
+		(at 253.365 41.275)
 		(diameter 0)
 		(color 0 0 0 0)
 	)
 	(junction
-		(at 253.365 41.275)
+		(at 175.006 78.3955)
 		(diameter 0)
 		(color 0 0 0 0)
@@
 	)
 	(junction
-		(at 175.006 78.359)
+		(at 164.846 88.519)
+		(diameter 0)
+		(color 0 0 0 0)
+	)
+	(junction
+		(at 175.006 80.9244)
 		(diameter 0)
 		(color 0 0 0 0)
@@
 	(wire
 		(pts
-			(xy 161.671 88.519) (xy 161.671 78.359)
+			(xy 164.846 80.9244) (xy 164.846 88.519)
 		)
 		(stroke
@@
 	(wire
 		(pts
-			(xy 164.846 80.899) (xy 164.846 88.519)
+			(xy 83.439 71.12) (xy 83.439 73.66)
 		)
 		(stroke
@@
 	(wire
 		(pts
-			(xy 83.439 71.12) (xy 83.439 73.66)
+			(xy 204.851 46.355) (xy 204.851 42.545)
 		)
 		(stroke
@@
 	(wire
 		(pts
-			(xy 204.851 46.355) (xy 204.851 42.545)
+			(xy 161.671 78.359) (xy 151.1046 78.359)
 		)
 		(stroke
@@
 	(wire
 		(pts
-			(xy 161.671 78.359) (xy 151.1046 78.359)
+			(xy 161.671 78.359) (xy 161.671 78.3955)
 		)
 		(stroke
@@
 	(wire
 		(pts
+			(xy 164.846 88.519) (xy 164.846 88.5444)
+		)
+		(stroke
+			(width 0)
+			(type default)
+		)
+	)
+	(wire
+		(pts
 			(xy 217.043 46.355) (xy 204.851 46.355)
 		)
@@
 	(wire
 		(pts
-			(xy 164.846 78.359) (xy 161.671 78.359)
+			(xy 151.1046 78.359) (xy 151.1046 78.9686)
 		)
 		(stroke
@@
 	(wire
 		(pts
-			(xy 151.1046 78.359) (xy 151.1046 78.9686)
+			(xy 245.237 36.195) (xy 245.237 31.115)
 		)
 		(stroke
@@
 	(wire
 		(pts
-			(xy 245.237 36.195) (xy 245.237 31.115)
+			(xy 164.846 78.3955) (xy 161.671 78.3955)
 		)
 		(stroke
@@
 	(wire
 		(pts
-			(xy 175.006 78.359) (xy 175.006 80.899)
+			(xy 175.006 78.3844) (xy 175.006 78.3955)
 		)
 		(stroke
@@
 	(wire
 		(pts
+			(xy 161.671 78.3955) (xy 161.671 88.519)
+		)
+		(stroke
+			(width 0)
+			(type default)
+		)
+	)
+	(wire
+		(pts
 			(xy 149.479 80.9244) (xy 149.479 81.7626)
 		)
@@
 	(wire
 		(pts
+			(xy 175.006 78.3955) (xy 175.006 80.9244)
+		)
+		(stroke
+			(width 0)
+			(type default)
+		)
+	)
+	(wire
+		(pts
 			(xy 84.201 78.74) (xy 85.979 78.74)
 		)
@@
 	(symbol
 		(lib_id "Jumper:Jumper_2_Open")
-		(at 169.926 80.899 0)
+		(at 169.926 80.9244 0)
 		(unit 1)
 		(exclude_from_sim no)
@@
 		(dnp no)
 		(property "Reference" "JP9"
-			(at 169.926 75.1037 0)
+			(at 169.926 75.1291 0)
 			(effects
 				(font
@@
 		)
 		(property "Value" "M/S"
-			(at 180.34 80.899 0)
+			(at 180.34 80.9244 0)
 			(effects
 				(font
@@
 		)
 		(property "Footprint" "Jumper:SolderJumper-2_P1.3mm_Open_Pad1.0x1.5mm"
-			(at 169.926 80.899 0)
+			(at 169.926 80.9244 0)
 			(effects
 				(font
@@
 		)
 		(property "Datasheet" "~"
-			(at 169.926 80.899 0)
+			(at 169.926 80.9244 0)
 			(effects
 				(font
@@
 		)
 		(property "Description" ""
-			(at 169.926 80.899 0)
+			(at 169.926 80.9244 0)
 			(effects
 				(font
@@
 	(symbol
 		(lib_id "Jumper:Jumper_2_Open")
-		(at 169.926 78.359 0)
+		(at 169.926 78.3955 0)
 		(unit 1)
 		(exclude_from_sim no)
@@
 		(dnp no)
 		(property "Reference" "JP8"
-			(at 169.926 72.5637 0)
+			(at 169.926 72.6002 0)
 			(effects
 				(font
@@
 		)
 		(property "Value" "CLK0"
-			(at 180.594 78.232 0)
+			(at 180.594 78.2685 0)
 			(effects
 				(font
@@
 		)
 		(property "Footprint" "Jumper:SolderJumper-2_P1.3mm_Open_Pad1.0x1.5mm"
-			(at 169.926 78.359 0)
+			(at 169.926 78.3955 0)
 			(effects
 				(font
@@
 		)
 		(property "Datasheet" "~"
-			(at 169.926 78.359 0)
+			(at 169.926 78.3955 0)
 			(effects
 				(font
@@
 		)
 		(property "Description" ""
-			(at 169.926 78.359 0)
+			(at 169.926 78.3955 0)
 			(effects
 				(font
@@
 	(symbol
 		(lib_id "power:GNDREF")
-		(at 175.006 80.899 90)
+		(at 175.006 80.9244 90)
 		(unit 1)
 		(exclude_from_sim no)
@@
 		(dnp no)
 		(property "Reference" "#PWR09"
-			(at 181.356 80.899 0)
+			(at 181.356 80.9244 0)
 			(effects
 				(font
@@
 		)
 		(property "Value" "GNDREF"
-			(at 178.943 83.693 90)
+			(at 178.943 83.7184 90)
 			(effects
 				(font
@@
 		)
 		(property "Footprint" ""
-			(at 175.006 80.899 0)
+			(at 175.006 80.9244 0)
 			(effects
 				(font
@@
 		)
 		(property "Datasheet" ""
-			(at 175.006 80.899 0)
+			(at 175.006 80.9244 0)
 			(effects
 				(font
@@
 		)
 		(property "Description" ""
-			(at 175.006 80.899 0)
+			(at 175.006 80.9244 0)
 			(effects
 				(font

Commit message: Kicad 9.0.5 update
Kicad update to 9.0.5
Src change: dtr is back, second buffer register added
Connections:
- net GNDREF: now also JP5.2 (B), JP6.2 (B), JP7.2 (B)
Changed lines of the file:
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@@
 (kicad_sch
-	(version 20231120)
+	(version 20250114)
 	(generator "eeschema")
-	(generator_version "8.0")
+	(generator_version "9.0")
 	(paper "A4")
 	(title_block
@@
 		(company "Victor A. Sergeev")
 	)
+	(text "mclk 512fs/32kHz = 16.384MHz  // current\nmclk 384fs/32kHz = 12.288MHz\nmclk 256fs/32kHz = 8.192MHz\nbck 24b/32kHz = 1.536MHz\nbck 16b/32kHz = 1.024MHz   // current\n\nCLK1 CLK0 MASTER CLOCK (MCLK) SELECTION\n0    0    128 fS\n0    1    256 fS\n1    0    384 fS\n1    1    512 fS // current\n\nFMT1 FMT0 FORMAT SELECTIONS\n0    0    24-Bit Left-Justified\n0    1    24-Bit I2S\n1    0    24-Bit Right-Justified\n1    1    16-Bit Right-Justified //current"
+		(exclude_from_sim no)
+		(at 222.504 164.338 0)
+		(effects
+			(font
+				(size 1.27 1.27)
+			)
+			(justify left bottom)
+		)
+	)
+	(text "4050 order\n14-15\n3-2\n5-4\n11-12\n7-6\n9-10"
+		(exclude_from_sim no)
+		(at 273.05 145.923 0)
+		(effects
+			(font
+				(size 1.27 1.27)
+			)
+			(justify left bottom)
+		)
+	)
+	(text "32KHz, 512fs, 16-bit Right Justified\nConsumer mode\n"
+		(exclude_from_sim no)
+		(at 84.709 35.052 0)
+		(effects
+			(font
+				(size 1.27 1.27)
+			)
+			(justify left bottom)
+		)
+	)
+	(text "When the DIT4192 is first powered up, the user must \nassert RST low in order to start the reset sequence. \nThe RST input must be low for a minimum of 500ns."
+		(exclude_from_sim no)
+		(at 222.25 129.032 0)
+		(effects
+			(font
+				(size 1.27 1.27)
+			)
+			(justify left bottom)
+		)
+	)
 	(junction
 		(at 161.671 78.3955)
@@
 	(wire
 		(pts
-			(xy 175.006 75.819) (xy 175.006 78.359)
-		)
-		(stroke
-			(width 0)
-			(type default)
-		)
-	)
-	(wire
-		(pts
 			(xy 239.903 46.355) (xy 248.539 46.355)
 		)
@@
 	(wire
 		(pts
-			(xy 175.006 78.3844) (xy 175.006 78.3955)
+			(xy 175.006 75.819) (xy 175.006 78.3955)
 		)
 		(stroke
@@
 		)
 	)
-	(text "mclk 512fs/32kHz = 16.384MHz  // current\nmclk 384fs/32kHz = 12.288MHz\nmclk 256fs/32kHz = 8.192MHz\nbck 24b/32kHz = 1.536MHz\nbck 16b/32kHz = 1.024MHz   // current\n\nCLK1 CLK0 MASTER CLOCK (MCLK) SELECTION\n0    0    128 fS\n0    1    256 fS\n1    0    384 fS\n1    1    512 fS // current\n\nFMT1 FMT0 FORMAT SELECTIONS\n0    0    24-Bit Left-Justified\n0    1    24-Bit I2S\n1    0    24-Bit Right-Justified\n1    1    16-Bit Right-Justified //current"
-		(exclude_from_sim no)
-		(at 222.504 164.338 0)
-		(effects
-			(font
-				(size 1.27 1.27)
-			)
-			(justify left bottom)
-		)
-	)
-	(text "4050 order\n14-15\n3-2\n5-4\n11-12\n7-6\n9-10"
-		(exclude_from_sim no)
-		(at 273.05 145.923 0)
-		(effects
-			(font
-				(size 1.27 1.27)
-			)
-			(justify left bottom)
-		)
-	)
-	(text "32KHz, 512fs, 16-bit Right Justified\nConsumer mode\n"
-		(exclude_from_sim no)
-		(at 84.709 35.052 0)
-		(effects
-			(font
-				(size 1.27 1.27)
-			)
-			(justify left bottom)
-		)
-	)
-	(text "When the DIT4192 is first powered up, the user must \nassert RST low in order to start the reset sequence. \nThe RST input must be low for a minimum of 500ns."
-		(exclude_from_sim no)
-		(at 222.25 129.032 0)
-		(effects
-			(font
-				(size 1.27 1.27)
-			)
-			(justify left bottom)
-		)
-	)
 	(global_label "CLK0"
 		(shape input)
@@
 		)
 		(property "Value" "MCLK_D"
-			(at 181.356 155.829 0)
+			(at 181.102 155.956 0)
 			(effects
 				(font
@@
 		(dnp no)
 		(property "Reference" "JP5"
-			(at 169.926 64.9437 0)
+			(at 169.926 70.358 0)
 			(effects
 				(font
@@
 		(dnp no)
 		(property "Reference" "JP7"
-			(at 169.926 70.0237 0)
+			(at 169.926 75.692 0)
 			(effects
 				(font
@@
 		(dnp no)
 		(property "Reference" "JP19"
-			(at 191.008 48.3403 0)
+			(at 197.866 41.402 0)
 			(effects
 				(font
@@
 		(dnp no)
 		(property "Reference" "JP9"
-			(at 169.926 75.1291 0)
+			(at 169.926 80.772 0)
 			(effects
 				(font
@@
 		(dnp no)
 		(property "Reference" "JP18"
-			(at 191.008 45.8003 0)
+			(at 197.866 38.862 0)
 			(effects
 				(font
@@
 		)
 		(property "Value" "BCK_D"
-			(at 180.975 143.383 0)
+			(at 180.086 143.51 0)
 			(effects
 				(font
@@
 		)
 		(property "Value" "WCLK_W"
-			(at 149.098 146.812 0)
+			(at 148.844 146.812 0)
 			(effects
 				(font
@@
 		(dnp no)
 		(property "Reference" "JP16"
-			(at 191.008 40.7203 0)
+			(at 197.866 33.274 0)
 			(effects
 				(font
@@
 		)
 		(property "Value" "MCLK_W"
-			(at 181.356 153.035 0)
+			(at 181.102 153.162 0)
 			(effects
 				(font
@@
 		(dnp no)
 		(property "Reference" "JP8"
-			(at 169.926 72.6002 0)
+			(at 169.926 78.232 0)
 			(effects
 				(font
@@
 		(dnp no)
 		(property "Reference" "JP17"
-			(at 191.008 43.2603 0)
+			(at 197.866 36.322 0)
 			(effects
 				(font
@@
 		)
 		(property "Value" "BCK_W"
-			(at 180.975 140.589 0)
+			(at 180.086 140.716 0)
 			(effects
 				(font
@@
 		(on_board yes)
 		(dnp no)
-		(fields_autoplaced yes)
 		(property "Reference" "R5"
-			(at 132.969 35.6575 90)
+			(at 132.842 38.1 90)
 			(effects
 				(font
@@
 		)
 		(property "Value" "300R"
-			(at 132.969 38.4326 90)
+			(at 133.096 40.64 90)
 			(effects
 				(font
@@
 		(dnp no)
 		(property "Reference" "JP6"
-			(at 169.926 67.4837 0)
+			(at 169.926 72.898 0)
 			(effects
 				(font
@@
 		)
 		(property "Value" "WCLK_D"
-			(at 149.098 149.606 0)
+			(at 148.844 149.606 0)
 			(effects
 				(font
@@
 		)
 	)
+	(embedded_fonts no)
 )
