File: hardware/MT32-DIT-v0.4/MT32-DIT-v0.4.kicad_sch (KiCad schematic)
At the start: 31 parts, among them J1 DEMUX_IN, J2 PWR_IN, J3 I2S_CONN, SW1 PWR, U1 4050, U10 PCM54HP, U2 4050, U3 4050, U4 Gowin9K, U5 4050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

Commit message: Kicad 9.0.5 update
Kicad update to 9.0.5
Src change: dtr is back, second buffer register added
Changed lines of the file:
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@@
 (kicad_sch
-	(version 20231120)
+	(version 20250114)
 	(generator "eeschema")
-	(generator_version "8.0")
+	(generator_version "9.0")
 	(paper "A4")
 	(title_block
@@
 		(company "Victor A. Sergeev")
 	)
+	(text "sum"
+		(exclude_from_sim no)
+		(at 38.608 37.846 0)
+		(effects
+			(font
+				(size 1.27 1.27)
+			)
+			(justify left bottom)
+		)
+	)
+	(text "f.back"
+		(exclude_from_sim no)
+		(at 36.068 40.386 0)
+		(effects
+			(font
+				(size 1.27 1.27)
+			)
+			(justify left bottom)
+		)
+	)
+	(text "offset"
+		(exclude_from_sim no)
+		(at 80.518 28.194 0)
+		(effects
+			(font
+				(size 1.27 1.27)
+			)
+			(justify left bottom)
+		)
+	)
+	(text "out"
+		(exclude_from_sim no)
+		(at 37.338 32.766 0)
+		(effects
+			(font
+				(size 1.27 1.27)
+			)
+			(justify left bottom)
+		)
+	)
+	(text "out"
+		(exclude_from_sim no)
+		(at 81.788 33.274 0)
+		(effects
+			(font
+				(size 1.27 1.27)
+			)
+			(justify left bottom)
+		)
+	)
+	(text "bank3"
+		(exclude_from_sim no)
+		(at 43.688 77.978 90)
+		(effects
+			(font
+				(size 1.27 1.27)
+			)
+			(justify left bottom)
+		)
+	)
+	(text "bank2"
+		(exclude_from_sim no)
+		(at 43.18 117.602 0)
+		(effects
+			(font
+				(size 1.27 1.27)
+			)
+			(justify right bottom)
+		)
+	)
+	(text "small noise reduction mod\n"
+		(exclude_from_sim no)
+		(at 41.148 191.262 0)
+		(effects
+			(font
+				(size 1.27 1.27)
+			)
+			(justify left bottom)
+		)
+	)
+	(text "bank1 3.3v\nbank2 3.3v\nbank3 1.8v"
+		(exclude_from_sim no)
+		(at 32.512 124.968 0)
+		(effects
+			(font
+				(size 1.27 1.27)
+			)
+			(justify left bottom)
+		)
+	)
+	(text "bank1"
+		(exclude_from_sim no)
+		(at 43.688 97.028 90)
+		(effects
+			(font
+				(size 1.27 1.27)
+			)
+			(justify left bottom)
+		)
+	)
+	(text "offset"
+		(exclude_from_sim no)
+		(at 36.068 27.686 0)
+		(effects
+			(font
+				(size 1.27 1.27)
+			)
+			(justify left bottom)
+		)
+	)
+	(text "bank1"
+		(exclude_from_sim no)
+		(at 43.434 65.278 0)
+		(effects
+			(font
+				(size 1.27 1.27)
+			)
+			(justify right bottom)
+		)
+	)
+	(text "bank2"
+		(exclude_from_sim no)
+		(at 31.496 89.408 90)
+		(effects
+			(font
+				(size 1.27 1.27)
+			)
+			(justify left bottom)
+		)
+	)
+	(text "f.back"
+		(exclude_from_sim no)
+		(at 80.518 40.894 0)
+		(effects
+			(font
+				(size 1.27 1.27)
+			)
+			(justify left bottom)
+		)
+	)
+	(text "sum"
+		(exclude_from_sim no)
+		(at 83.058 38.354 0)
+		(effects
+			(font
+				(size 1.27 1.27)
+			)
+			(justify left bottom)
+		)
+	)
+	(text "bank1"
+		(exclude_from_sim no)
+		(at 31.496 116.078 90)
+		(effects
+			(font
+				(size 1.27 1.27)
+			)
+			(justify left bottom)
+		)
+	)
 	(junction
 		(at 139.954 190.754)
@@
 		)
 	)
-	(text "sum"
-		(exclude_from_sim no)
-		(at 38.608 37.846 0)
-		(effects
-			(font
-				(size 1.27 1.27)
-			)
-			(justify left bottom)
-		)
-	)
-	(text "f.back"
-		(exclude_from_sim no)
-		(at 36.068 40.386 0)
-		(effects
-			(font
-				(size 1.27 1.27)
-			)
-			(justify left bottom)
-		)
-	)
-	(text "offset"
-		(exclude_from_sim no)
-		(at 80.518 28.194 0)
-		(effects
-			(font
-				(size 1.27 1.27)
-			)
-			(justify left bottom)
-		)
-	)
-	(text "out"
-		(exclude_from_sim no)
-		(at 37.338 32.766 0)
-		(effects
-			(font
-				(size 1.27 1.27)
-			)
-			(justify left bottom)
-		)
-	)
-	(text "out"
-		(exclude_from_sim no)
-		(at 81.788 33.274 0)
-		(effects
-			(font
-				(size 1.27 1.27)
-			)
-			(justify left bottom)
-		)
-	)
-	(text "bank3"
-		(exclude_from_sim no)
-		(at 43.688 77.978 90)
-		(effects
-			(font
-				(size 1.27 1.27)
-			)
-			(justify left bottom)
-		)
-	)
-	(text "bank2"
-		(exclude_from_sim no)
-		(at 43.18 117.602 0)
-		(effects
-			(font
-				(size 1.27 1.27)
-			)
-			(justify right bottom)
-		)
-	)
-	(text "small noise reduction mod\n"
-		(exclude_from_sim no)
-		(at 41.148 191.262 0)
-		(effects
-			(font
-				(size 1.27 1.27)
-			)
-			(justify left bottom)
-		)
-	)
-	(text "bank1 3.3v\nbank2 3.3v\nbank3 1.8v"
-		(exclude_from_sim no)
-		(at 32.512 124.968 0)
-		(effects
-			(font
-				(size 1.27 1.27)
-			)
-			(justify left bottom)
-		)
-	)
-	(text "bank1"
-		(exclude_from_sim no)
-		(at 43.688 97.028 90)
-		(effects
-			(font
-				(size 1.27 1.27)
-			)
-			(justify left bottom)
-		)
-	)
-	(text "offset"
-		(exclude_from_sim no)
-		(at 36.068 27.686 0)
-		(effects
-			(font
-				(size 1.27 1.27)
-			)
-			(justify left bottom)
-		)
-	)
-	(text "bank1"
-		(exclude_from_sim no)
-		(at 43.434 65.278 0)
-		(effects
-			(font
-				(size 1.27 1.27)
-			)
-			(justify right bottom)
-		)
-	)
-	(text "bank2"
-		(exclude_from_sim no)
-		(at 31.496 89.408 90)
-		(effects
-			(font
-				(size 1.27 1.27)
-			)
-			(justify left bottom)
-		)
-	)
-	(text "f.back"
-		(exclude_from_sim no)
-		(at 80.518 40.894 0)
-		(effects
-			(font
-				(size 1.27 1.27)
-			)
-			(justify left bottom)
-		)
-	)
-	(text "sum"
-		(exclude_from_sim no)
-		(at 83.058 38.354 0)
-		(effects
-			(font
-				(size 1.27 1.27)
-			)
-			(justify left bottom)
-		)
-	)
-	(text "bank1"
-		(exclude_from_sim no)
-		(at 31.496 116.078 90)
-		(effects
-			(font
-				(size 1.27 1.27)
-			)
-			(justify left bottom)
-		)
-	)
 	(label "PCM27"
 		(at 93.218 21.844 0)
-		(fields_autoplaced yes)
 		(effects
 			(font
@@
 	(label "PCM23"
 		(at 93.218 32.004 0)
-		(fields_autoplaced yes)
 		(effects
 			(font
@@
 	(label "PCM20"
 		(at 48.768 39.116 0)
-		(fields_autoplaced yes)
 		(effects
 			(font
@@
 	(label "PCM25"
 		(at 48.768 26.416 0)
-		(fields_autoplaced yes)
 		(effects
 			(font
@@
 	(label "PCM26"
 		(at 97.536 24.384 0)
-		(fields_autoplaced yes)
 		(effects
 			(font
@@
 	(label "PCM26"
 		(at 48.768 23.876 0)
-		(fields_autoplaced yes)
 		(effects
 			(font
@@
 	(label "PCM27"
 		(at 48.768 21.336 0)
-		(fields_autoplaced yes)
 		(effects
 			(font
@@
 	(label "PCM27"
 		(at 46.482 182.88 270)
-		(fields_autoplaced yes)
 		(effects
 			(font
@@
 	(label "PCM1"
 		(at 64.008 19.304 180)
-		(fields_autoplaced yes)
 		(effects
 			(font
@@
 	(label "PCM1"
 		(at 19.558 18.796 180)
-		(fields_autoplaced yes)
 		(effects
 			(font
@@
 	(label "PCM19"
 		(at 93.218 42.164 0)
-		(fields_autoplaced yes)
 		(effects
 			(font
@@
 	(label "PCM23"
 		(at 48.768 31.496 0)
-		(fields_autoplaced yes)
 		(effects
 			(font
@@
 	(label "GNDREF"
 		(at 97.536 34.544 0)
-		(fields_autoplaced yes)
 		(effects
 			(font
@@
 	(label "PCM1"
 		(at 35.052 171.45 180)
-		(fields_autoplaced yes)
 		(effects
 			(font
@@
 	(label "PCM28"
 		(at 93.218 19.304 0)
-		(fields_autoplaced yes)
 		(effects
 			(font
@@
 	(label "PCM21"
 		(at 48.768 36.576 0)
-		(fields_autoplaced yes)
 		(effects
 			(font
@@
 	(label "PCM28"
 		(at 57.912 171.45 0)
-		(fields_autoplaced yes)
 		(effects
 			(font
@@
 	(label "PCM25"
 		(at 93.218 26.924 0)
-		(fields_autoplaced yes)
 		(effects
 			(font
@@
 	(label "PCM20"
 		(at 93.218 39.624 0)
-		(fields_autoplaced yes)
 		(effects
 			(font
@@
 	(label "PCM19"
 		(at 48.768 41.656 0)
-		(fields_autoplaced yes)
 		(effects
 			(font
@@
 	(label "GNDREF"
 		(at 48.768 34.036 0)
-		(fields_autoplaced yes)
 		(effects
 			(font
@@
 	(label "PCM21"
 		(at 93.218 37.084 0)
-		(fields_autoplaced yes)
 		(effects
 			(font
@@
 	(label "PCM28"
 		(at 48.768 18.796 0)
-		(fields_autoplaced yes)
 		(effects
 			(font
@@
 		)
 	)
+	(embedded_fonts no)
 )

Commit message: HW updates
Service notes 2nd and 3rd editions added. Kicad schematic update - LSB bit route can be selected for external input.
Parts:
- added J4: LSB, Connector_PinHeader_2.54mm:PinHeader_1x01_P2.54mm_Vertical, symbol Connector:Conn_01x01_Socket
- added J5: LSB_conn, Connector_PinHeader_2.54mm:PinHeader_1x03_P2.54mm_Vertical, symbol Connector:Conn_01x03_Socket
- added J6: GND hook, Connector_PinHeader_2.54mm:PinHeader_1x03_P2.54mm_Vertical, symbol Connector:Conn_01x03_Socket
Connections:
- net GNDREF: now also J6.1 (Pin_1), J6.2 (Pin_2), J6.3 (Pin_3)
- net P16: now also J5.1 (Pin_1); no longer U5.11
- new net: J4.1 (Pin_1), J5.3 (Pin_3)
- new net LSB: J5.2 (Pin_2), U5.11
